Commit message: fix : Updated urdf files to add new stl file, resize robot.

File: catkin_ws/src/my_robot/urdf/diff_bot/accessories/depth_camera.urdf.xacro (robot description, xacro)
@@ -5,5 +5,5 @@
   <xacro:macro name="sensor_kinect" params="parent">
     <joint name="camera_rgb_joint" type="fixed">
-      <origin xyz="0.6 0 0.06" rpy="0 0 0"/>
+      <origin xyz="0.3 0 0.09" rpy="0 0 0"/>
       <parent link="${parent}"/>
       <child link="camera_rgb_frame" />
@@ -25,5 +25,5 @@
        <origin xyz="0 0 0" rpy="0 0 0"/>
         <geometry>
-         <mesh filename="package://my_robot/meshes/kinect.dae"/>
+         <mesh filename="package://my_robot/meshes/kinect.stl"/>
         </geometry>
         <material name="Blue" />
@@ -32,5 +32,5 @@
         <origin xyz="0.0 0.0 0.0" rpy="0 0 0"/>
   	    <geometry>
-  	      <box size="0.07271 0.27794 0.073"/>
+         <mesh filename="package://my_robot/meshes/kinect.stl"/>
   	    </geometry>
   	  </collision>
@@ -57,4 +57,5 @@
 	<!-- Kinect sensor for simulation -->
     <gazebo reference="camera_link">
+      <material value="Gazebo/Red" />
       <sensor type="depth" name="camera">
         <always_on>true</always_on>

File: catkin_ws/src/my_robot/urdf/diff_bot/accessories/sick_s300.urdf.xacro (robot description, xacro)
@@ -24,5 +24,5 @@
       <sensor type="ray" name="${prefix}${link}">
         <pose>0 0 0 0 0 0</pose>
-        <visualize>false</visualize>
+        <visualize>true</visualize>
         <update_rate>12.5</update_rate>
         <ray>

File: catkin_ws/src/my_robot/urdf/diff_bot/skid_steer_base.urdf.xacro (robot description, xacro)
@@ -4,13 +4,13 @@
     <xacro:include filename="$(find my_robot)/urdf/diff_bot/common_properties.urdf.xacro" />
     <!-- Define a number of dimensions using properties -->
-    <xacro:property name="base_size_x" value="1.20" />
-    <xacro:property name="base_size_y" value="1.0" />
-    <xacro:property name="base_size_z" value="0.26191" />
-    <xacro:property name="wheel_length" value="0.07032" />
+    <xacro:property name="base_size_x" value="0.6" />
+    <xacro:property name="base_size_y" value="0.5" />
+    <xacro:property name="base_size_z" value="0.130955" />
+    <xacro:property name="wheel_length" value="0.03516" />
     <!-- 0.06032 value for perfect fit.-->
-    <xacro:property name="wheel_radius" value="0.17" />
-    <xacro:property name="wheel_offset_x" value="0.6" />
-    <xacro:property name="wheel_offset_y" value="0.46984" />
-    <xacro:property name="wheel_offset_z" value="-0.045955" />
+    <xacro:property name="wheel_radius" value="0.085" />
+    <xacro:property name="wheel_offset_x" value="0.3" />
+    <xacro:property name="wheel_offset_y" value="0.23492" />
+    <xacro:property name="wheel_offset_z" value="-0.0229775" />
     <xacro:property name="PI" value="3.1415" />
     <!-- differential_drive_controller update rate -->
@@ -136,5 +136,5 @@
     <gazebo>
         <plugin name="skid_steer_drive_controller" filename="libgazebo_ros_skid_steer_drive.so">
-            <updateRate>30.0</updateRate>
+            <updateRate>90.0</updateRate>
             <robotNamespace>/my_robot</robotNamespace>
             <leftFrontJoint>base_fl_wheel_joint</leftFrontJoint>
